Commit message: Update URDF, launch files and add config folder for elder_robot

File: urdf/elderbot.urdf (robot description, URDF)
Before this commit: robot elderbot, 8 links, 7 joints
Joints:
- joint base_footprint_joint: origin xyz=0 0 0 rpy=0 0 0 -> xyz=0 0 0.152 rpy=0 0 0

File: urdf/elderbot.urdf.xacro (robot description, xacro)
@@ -4,18 +4,24 @@
   <gazebo>
     <plugin name="diff_drive" filename="libgazebo_ros_diff_drive.so">
+      <update_rate>10</update_rate>
       <left_joint>left_rear_wheel_joint</left_joint>
       <right_joint>right_rear_wheel_joint</right_joint>
       <wheel_separation>${wheel_separation}</wheel_separation>
       <wheel_diameter>${wheel_radius * 2}</wheel_diameter>
+      <max_wheel_torque>20</max_wheel_torque>
+      <max_wheel_acceleration>1.0</max_wheel_acceleration>
+      <commandTopic>cmd_vel</commandTopic>
+      <odometryTopic>odom</odometryTopic>
+      <publishOdomTF>true</publishOdomTF>
+      <odometry_frame>odom</odometry_frame>
+      <robot_base_frame>base_footprint</robot_base_frame>
+      <publish_odom>true</publish_odom>
+      <publish_odom_tf>true</publish_odom_tf>
+      <publish_wheel_tf>false</publish_wheel_tf>
       <ros>
-        <remapping>cmd_vel:=/cmd_vel</remapping>
-        <remapping>odom:=/odom</remapping>
+          <namespace>/</namespace>
+          <remapping>cmd_vel:=cmd_vel</remapping>
+          <remapping>odom:=odom</remapping>
       </ros>
-      <odometryFrame>odom</odometryFrame>
-      <robotBaseFrame>base_link</robotBaseFrame>
-      <publishOdom>true</publishOdom>
-      <publishTf>true</publishTf>
-      <publishWheelJointState>true</publishWheelJointState>
-      <legacyMode>false</legacyMode>
     </plugin>
     <plugin name="joint_state_publisher" filename="libgazebo_ros_joint_state_publisher.so">

File: urdf/robotcore.xacro (robot description, xacro)
@@ -21,5 +21,5 @@
         <parent link="base_footprint"/>
         <child link="base_link"/>
-        <origin xyz="0 0 0" rpy="0 0 0"/>
+        <origin xyz="0 0 0.152" rpy="0 0 0"/>
     </joint>
     <!-- CHASSIS -->

File: urdf/sensors.xacro (robot description, xacro)
@@ -33,5 +33,5 @@
                         <min_angle>-3.14</min_angle>
                         <max_angle>3.14</max_angle>
-                    </horizontal>
+                    </horizontal>S
                 </scan>
                 <range>
@@ -46,5 +46,5 @@
                 </ros>
                 <output_type>sensor_msgs/LaserScan</output_type>
-                <frameName>lidar_frame</frameName>
+                <frameName>laser_frame</frameName>
             </plugin>
         </sensor>
